Commit message: [cnoid,description] Update SampleField.

File: description/urdf/SampleField.urdf (robot description, URDF)
Before this commit: robot SampleField, 3 links, 2 joints
Links:
- added link HandleRightHand1, mass 1e-06; visual box size=0.2 0.2 0.02
- link HandleLeftHand1: geometry visual cylinder length=0.15 radius=0.015
Joints:
- added joint HandleRightHand1: type fixed, parent Root, child HandleRightHand1, origin xyz=1.4 -0.7 1.0 rpy=-1.57079632679 -0.0 0.0
- joint HandleLeftHand1: origin xyz=0.9 0.5 0.9 rpy=-2.35619449019 -0.0 0.0 -> xyz=0.9 0.5 0.8 rpy=-2.35619449019 -0.0 0.0

Commit message: Update SampleField.

File: description/urdf/SampleField.urdf (robot description, URDF)
Before this commit: robot SampleField, 4 links, 3 joints
Joints:
- joint HandleLeftHand1: origin xyz=0.9 0.5 0.8 rpy=-2.35619449019 -0.0 0.0 -> xyz=0.9 0.5 0.8 rpy=0.5235987755982988 -0.0 0.0

Commit message: [CI] walk two more steps forward and jump.

File: description/urdf/SampleField.urdf (robot description, URDF)
Before this commit: robot SampleField, 4 links, 3 joints
Joints:
- joint HandleRightHand1: origin xyz=1.4 -0.7 1.0 rpy=-1.57079632679 -0.0 0.0 -> xyz=1.8 -0.7 1.0 rpy=-1.57079632679 -0.0 0.0

Commit message: Add collision tags to SampleField.urdf

File: description/urdf/SampleField.urdf (robot description, URDF)
Before this commit: robot SampleField, 4 links, 3 joints
Links:
- link HandleLeftHand1: geometry collision cylinder length=0.15 radius=0.015; visual cylinder length=0.15 radius=0.015
- link HandleRightHand1: geometry collision box size=0.2 0.2 0.02; visual box size=0.2 0.2 0.02
- link StepRightFoot1: geometry collision box size=0.2 0.2 0.02; visual box size=0.2 0.2 0.02

Commit message: [cnoid,description] Delete unnecessary transformation in the handle.

File: description/urdf/SampleField.urdf (robot description, URDF)
Before this commit: robot SampleField, 4 links, 3 joints
Joints:
- joint HandleLeftHand1: origin xyz=0.9 0.5 0.8 rpy=0.5235987755982988 -0.0 0.0 -> xyz=0.9 0.5 0.8 rpy=0.0 -0.0 0.0

Commit message: [description] Add SampleStepladder.urdf

File: description/urdf/SampleField.urdf (robot description, URDF)
Before this commit: robot SampleField, 4 links, 3 joints
Links:
- link Root: mass 1e-06 -> None
