Commit message: [cnoid, description] Update ampleStepladder.

File: description/urdf/SampleStepladder.urdf (robot description, URDF)
Before this commit: robot SampleStepladder, 8 links, 7 joints
Links:
- removed link Step5
- link HandrailLeft: geometry visual box size=0.02 2.0 0.02
- link HandrailRight: geometry visual box size=0.02 2.0 0.02
Joints:
- removed joint Step5
